Commit message: fix(3d-replay): correct gripper range mapping
Map normalized gripper commands through each loaded URDF limit.
Correct TacCap mimic direction and constrain each finger to 29.235 degrees.

File: public/urdf/taccap-grippers/left/gripper.urdf (robot description, URDF)
Before this commit: robot taccap_left_gripper, 5 links, 4 joints
Joints:
- joint joint1: limit lower=0 upper=1 effort=1 velocity=1 -> lower=0 upper=0.5102470068205421 effort=1 velocity=1; mimic joint=joint2 multiplier=-1 offset=0 -> (none)
- joint joint2: limit lower=-1 upper=0 effort=1 velocity=1 -> lower=-0.5102470068205421 upper=0 effort=1 velocity=1; mimic (none) -> joint=joint1 multiplier=-1 offset=0

File: public/urdf/taccap-grippers/right/gripper.urdf (robot description, URDF)
Before this commit: robot taccap_right_gripper, 5 links, 4 joints
Joints:
- joint joint1: limit lower=0 upper=1 effort=1 velocity=1 -> lower=0 upper=0.5102470068205421 effort=1 velocity=1; mimic joint=joint2 multiplier=-1 offset=0 -> (none)
- joint joint2: limit lower=-1 upper=0 effort=1 velocity=1 -> lower=-0.5102470068205421 upper=0 effort=1 velocity=1; mimic (none) -> joint=joint1 multiplier=-1 offset=0

Commit message: fix(taccap): set finger limit to 28.92 degrees
Apply the corrected single-finger travel to both URDFs and keep the
regression expectation aligned.

File: public/urdf/taccap-grippers/left/gripper.urdf (robot description, URDF)
Before this commit: robot taccap_left_gripper, 5 links, 4 joints
Joints:
- joint joint1: limit lower=0 upper=0.5102470068205421 effort=1 velocity=1 -> lower=0 upper=0.5047492196767601 effort=1 velocity=1
- joint joint2: limit lower=-0.5102470068205421 upper=0 effort=1 velocity=1 -> lower=-0.5047492196767601 upper=0 effort=1 velocity=1

File: public/urdf/taccap-grippers/right/gripper.urdf (robot description, URDF)
Before this commit: robot taccap_right_gripper, 5 links, 4 joints
Joints:
- joint joint1: limit lower=0 upper=0.5102470068205421 effort=1 velocity=1 -> lower=0 upper=0.5047492196767601 effort=1 velocity=1
- joint joint2: limit lower=-0.5102470068205421 upper=0 effort=1 velocity=1 -> lower=-0.5047492196767601 upper=0 effort=1 velocity=1
